File: PowerMeter.sch (KiCad schematic (older format))
At the start: 16 parts, among them P1 SERIAL, SW1 FLASH, U1 ESP-01, U2 PC817

Commit message: Correct pushbutton
Parts:
- removed SW?: FLASH, symbol SW_PUSH
- U1, U?: symbol ESP-01v090 -> ESP-01v090-RESCUE-PowerMeter
Changed lines of the file:
@@
 EESchema Schematic File Version 2
+LIBS:PowerMeter-rescue
 LIBS:power
 LIBS:device
@@
 	7400 4200 8550 4200
 $Comp
-L ESP-01v090 U1
+L ESP-01v090-RESCUE-PowerMeter U1
 U 1 1 5A204CCD
 P 4850 3650
@@
 $EndComp
 $Comp
-L ESP-01v090 U?
+L ESP-01v090-RESCUE-PowerMeter U?
 U 1 1 5A207F02
 P 4850 3650
@@
 	1    0    0    -1
 $EndComp
-$Comp
-L SW_PUSH SW?
-U 1 1 5A207F0B
-P 6200 2600
-F 0 "SW?" H 6350 2710 50  0000 C CNN
-F 1 "FLASH" H 6200 2520 50  0000 C CNN
-F 2 "" H 6200 2600 50  0000 C CNN
-F 3 "" H 6200 2600 50  0000 C CNN
-	1    6200 2600
-	1    0    0    -1
-$EndComp
